Commit message: two finish

File: install/modelo_robot/share/modelo_robot/urdf/URDF_Microproyecto_9.urdf (robot description, URDF)
Before this commit: robot URDF_Microproyecto_9, 4 links, 3 joints
Links:
- link Cam_link: geometry collision box size=0.025 0.025 0.015; visual mesh filename=package://modelo_robot/meshes/Cam_link.STL
- link Rueda_der: geometry collision cylinder length=0.012 radius=0.015; visual mesh filename=package://modelo_robot/meshes/Rueda_der.STL
- link Rueda_izq: geometry collision cylinder length=0.012 radius=0.015; visual mesh filename=package://modelo_robot/meshes/Rueda_izq.STL
- link base_link: geometry collision box size=0.12 0.085 0.05; visual mesh filename=package://modelo_robot/meshes/base_link.STL

Commit message: 3er commit

File: install/modelo_robot/share/modelo_robot/urdf/URDF_Microproyecto_9.urdf (robot description, URDF)
Before this commit: robot URDF_Microproyecto_9, 4 links, 3 joints
Joints:
- joint joint_izq: axis 0 0 1 -> 0 0 -1

Commit message: feat: Gazebo Ignition + micro-ROS + joy_controller Xbox

File: install/modelo_robot/share/modelo_robot/urdf/URDF_Microproyecto_9.urdf (robot description, URDF)
Before this commit: robot URDF_Microproyecto_9, 4 links, 3 joints
Joints:
- joint joint_der: axis 0 0 -1 -> 0 0 1
- joint joint_izq: axis 0 0 -1 -> 0 0 1

Commit message: agrega modelo URDF

File: install/modelo_robot/share/modelo_robot/urdf/URDF_Microproyecto_9.urdf (robot description, URDF)
Before this commit: robot URDF_Microproyecto_9, 4 links, 3 joints
Links:
- link Cam_link: mass 0.00241389293196676 -> 0.001
- link base_link: mass 0.476441238351147 -> 0.47644

Commit message: adelante y atras bien

File: install/modelo_robot/share/modelo_robot/urdf/URDF_Microproyecto_9.urdf (robot description, URDF)
Before this commit: robot URDF_Microproyecto_9, 4 links, 3 joints
Joints:
- joint joint_der: origin xyz=-0.034252 -0.040164 -0.0010202 rpy=1.5708 0 0 -> xyz=-0.034252 -0.040164 -0.0010202 rpy=-1.5708 0 0
